File: main/explorekb75/explorekb75.kicad_sch (KiCad schematic)
At the start: 1 part, among them U1 YAAJ_WeAct_BlackPill_Part_Like

Commit message: added init board and pcb
Parts:
- added J?: Conn_01x04, symbol Connector_Generic:Conn_01x04
- added R1, R2: 4k7, _scott_lib:C_0603_1608Metric_Pad1.08x0.95mm_HandSolder, symbol Device:R
- added U2: SSD1306, _scott_lib:SSD1306_128X32, symbol _scott_lib:SSD1306
Connections:
- net COL 0: now also U1.32 (PA6); no longer U1.36 (PB2)
- net COL 1: now also U1.31 (PA5); no longer U1.35 (PB1)
- net COL 10: now also U1.4 (PB15); no longer U1.2 (PB13)
- net COL 11: now also U1.5 (PA8); no longer U1.4 (PB15)
- net COL 12: now also U1.10 (PA15); no longer U1.5 (PA8)
- net COL 13: now also U1.12 (PB4); no longer U1.13 (PB5)
- net COL 2: now also U1.30 (PA4); no longer U1.34 (PB0)
- net COL 3: now also U1.29 (PA3); no longer U1.33 (PA7)
- net COL 4: now also U1.28 (PA2); no longer U1.32 (PA6)
- net COL 5: now also U1.26 (PA0); no longer U1.31 (PA5)
- net COL 6: now also U1.24 (PC15); no longer U1.30 (PA4)
- net COL 7: now also U1.23 (PC14); no longer U1.28 (PA2)
- net COL 8: now also U1.1 (PB12); no longer U1.27 (PA1)
- net COL 9: now also U1.3 (PB14); no longer U1.1 (PB12)
- net GND: now also J?.4 (Pin_4), U2.4 (GND)
- net ROW 0: now also U1.33 (PA7); no longer U1.37 (PB10)
- net ROW 1: now also U1.27 (PA1); no longer U1.29 (PA3)
- net ROW 2: now also U1.16 (PB8); no longer U1.26 (PA0)
- net ROW 3: now also U1.13 (PB5); no longer U1.3 (PB14)
- net ROW 5: now also U1.2 (PB13); no longer U1.12 (PB4)
- net SCL1: now reaches U1.14 (PB6)
- net SCL1: now also R2.2, U2.2 (SCK)
- net SDA1: now reaches U1.15 (PB7)
- net SDA1: now also R1.2, U2.1 (SDA)
- net +3V3: now reaches U1.20 (3V3)
- net +3V3: now also J?.3 (Pin_3), R1.1, R2.1, U2.3 (VCC)
- net UART1_TX: now reaches U1.6 (PA9)
- net UART1_TX: now also J?.1 (Pin_1)
- net UART1_RX: now reaches U1.7 (PA10)
- net UART1_RX: now also J?.2 (Pin_2)
- new net ROT1_A: U1.35 (PB1)
- new net ROT1_B: U1.34 (PB0)
- new net ROT2_A: U1.37 (PB10)
- new net ROT2_B: U1.36 (PB2)
- no-connect marks 17 -> 8
Other:
- sheet Key Matrix ports: added ROT1_A, ROT1_B, ROT2_A, ROT2_B; removed none
- moved on the sheet: U1
