File: main/explorekb75/key_matrix.kicad_sch (KiCad schematic)
At the start: 119 parts, among them SW1 SW_SPST, SW10 SW_SPST, SW11 SW_SPST, SW12 SW_SPST, SW13 SW_SPST, SW14 SW_SPST, SW15 SW_SPST, SW16 SW_SPST, SW17 SW_SPST, SW18 SW_SPST, SW19 SW_SPST, SW2 SW_SPST, SW20 SW_SPST, SW21 SW_SPST, SW22 SW_SPST, SW23 SW_SPST, SW24 SW_SPST, SW25 SW_SPST, SW26 SW_SPST, SW27 SW_SPST, SW28 SW_SPST, SW29 SW_SPST, SW3 SW_SPST, SW30 SW_SPST, SW31 SW_SPST, SW32 SW_SPST, SW33 SW_SPST, SW34 SW_SPST, SW35 SW_SPST, SW36 SW_SPST, SW37 SW_SPST, SW38 SW_SPST, SW39 SW_SPST, SW4 SW_SPST, SW40 SW_SPST, SW41 SW_SPST, SW42 SW_SPST, SW43 SW_SPST, SW44 SW_SPST, SW45 SW_SPST, SW46 SW_SPST, SW47 SW_SPST, SW48 SW_SPST, SW49 SW_SPST, SW5 SW_SPST, SW50 SW_SPST, SW51 SW_SPST, SW52 SW_SPST, SW53 SW_SPST, SW54 SW_SPST, SW55 SW_SPST, SW56 SW_SPST, SW57 SW_SPST, SW58 SW_SPST, SW59 SW_SPST, SW6 SW_SPST, SW60 SW_SPST, SW61 SW_SPST, SW62 SW_SPST, SW63 SW_SPST, SW64 SW_SPST, SW65 SW_SPST, SW66 SW_SPST, SW67 SW_SPST, SW68 SW_SPST, SW69 SW_SPST, SW7 SW_SPST, SW70 SW_SPST, SW71 SW_SPST, SW72 SW_SPST, SW73 SW_SPST, SW74 SW_SPST, SW75 SW_SPST, SW76 SW_SPST, SW77 SW_SPST, SW78 SW_SPST, SW79 SW_SPST, SW8 SW_SPST, SW9 SW_SPST

Commit message: added init board and pcb
Parts:
- removed SW14, SW15: SW_SPST, keyswitch_pretty:Kailh_socket_MX, symbol Switch:SW_SPST
- added C1, C2, C3, C4: 100n, _scott_lib:C_0603_1608Metric_Pad1.08x0.95mm_HandSolder, symbol Device:C
- added SW14, SW15: RotaryEncoder_Switch, _scott_lib:RotaryEncoder_Alps_EC11E-Switch_Vertical_H20mm, symbol Device:RotaryEncoder_Switch
- D1, D10, D11, D12, D13, D14, D15, D16, D17, D18, D19, D2, D20, D21, D22, D23, D24, D25, D26, D27, D28, D29, D3, D30, D31, D32, D33, D34, D35, D36, D37, D38, D39, D4, D40, D5, D6, D7, D8, D9: footprint Package_TO_SOT_SMD:SOT-23 -> _scott_lib:SOT-23
Connections:
- net COL 13: now also SW14.S2, SW15.S1
- net ROT1_2: now reaches D7.1
- net ROT1_2: now also SW14.S1
- net ROT2_2: now reaches D28.2
- net ROT2_2: now also SW15.S2
- net at D35.1: now also SW69.1 (A)
- net at D35.2: no longer SW69.1 (A)
- new net GND: C1.2, C2.2, C3.2, C4.2, SW14.C, SW15.C
- new net ROT1_A: C1.1, SW14.B
- new net ROT1_B: C2.1, SW14.A
- new net ROT2_A: C3.1, SW15.B
- new net ROT2_B: C4.1, SW15.A
Other:
- moved on the sheet: D1, D10, D11, D12, D13, D14, D15, D16, D17, D18, D19, D2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
