File: main/explorekb75-rev4/explorekb75s.kicad_sch (KiCad schematic)
At the start: 5 parts, among them J1 Conn_01x04, U1 YAAJ_WeAct_BlackPill_Part_Like, U2 SSD1306

Commit message: complete wiring for rev 4
Connections:
- net COL 7: now also U1.1 (PB12); no longer U1.23 (PC14)
- net COL 8: now also U1.23 (PC14); no longer U1.1 (PB12)
Changed lines of the file:
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@@
-    (effects (font (size 1.27 1.27)) (justify right bottom))
-  )
-  (label "COL 7" (at 133.35 107.95 180)
     (effects (font (size 1.27 1.27)) (justify right bottom))
   )
@@
     (effects (font (size 1.27 1.27)) (justify right bottom))
   )
-  (label "COL 8" (at 189.23 64.77 0)
+  (label "COL 8" (at 133.35 107.95 180)
+    (effects (font (size 1.27 1.27)) (justify right bottom))
+  )
+  (label "COL 7" (at 189.23 64.77 0)
     (effects (font (size 1.27 1.27)) (justify left bottom))
   )
