File: hardware/keyboard pcb/explorekb75-rev4/explorekb75s.kicad_sch (KiCad schematic)
At the start: 5 parts, among them J1 Conn_01x04, U1 YAAJ_WeAct_BlackPill_Part_Like, U2 SSD1306

Commit message: refactored paths
Parts:
- removed U1: YAAJ_WeAct_BlackPill_Part_Like, YAAJ_Blackpill:YAAJ_WeAct_BlackPill_2, symbol YAAJ_WeAct_BlackPill_Part_Like:YAAJ_WeAct_BlackPill_Part_Like
- added U1: WeAct_BlackPill, scottcjx-keyboard_components:WeAct_BlackPill_2, symbol scottcjx-keyboard_components:WeAct_BlackPill
- R1, R2: footprint _scott_lib:C_0603_1608Metric_Pad1.08x0.95mm_HandSolder -> scottcjx-keyboard_components:C_0603
- U2: footprint _scott_lib:SSD1306_128X32 -> scottcjx-keyboard_components:SSD1306_128X32
Connections:
- net +3V3: now also U1.20 (3V3)
- net COL 0: now also U1.32 (PA6)
- net COL 1: now also U1.31 (PA5)
- net COL 10: now also U1.4 (PB15)
- net COL 11: now also U1.5 (PA8)
- net COL 12: now also U1.10 (PA15)
- net COL 13: now also U1.12 (PB4)
- net COL 2: now also U1.30 (PA4)
- net COL 3: now also U1.29 (PA3)
- net COL 4: now also U1.28 (PA2)
- net COL 5: now also U1.26 (PA0)
- net COL 6: now also U1.24 (PC15)
- net COL 7: now also U1.1 (PB12)
- net COL 8: now also U1.23 (PC14)
- net COL 9: now also U1.3 (PB14)
- net GND: now also U1.19 (GND), U1.39 (GND)
- net ROT1_A: now also U1.35 (PB1)
- net ROT1_B: now also U1.34 (PB0)
- net ROT2_A: now also U1.37 (PB10)
- net ROT2_B: now also U1.36 (PB2)
- net ROW 0: now also U1.33 (PA7)
- net ROW 1: now also U1.27 (PA1)
- net ROW 2: now also U1.16 (PB8)
- net ROW 3: now also U1.13 (PB5)
- net ROW 4: now also U1.11 (PB3)
- net ROW 5: now also U1.2 (PB13)
- net SCL1: now also U1.14 (PB6)
- net SDA1: now also U1.15 (PB7)
- net UART1_RX: now also U1.7 (PA10)
- net UART1_TX: now also U1.6 (PA9)
- net ~{RST}: now also U1.25 (RES)
